File: can-transceiver-board.kicad_pcb (KiCad board)
At the start: 2 copper layers, 20 x 13 mm, 6 parts, among them K1 JMP, P1 CONN_5, U1 MAX3051

Commit message: Add text to silkscreen, increased power tracks.
Routing:
- net GND: track 32.6 -> 53.2 mm
- net Net-(CONN1-Pad1): track 8.50 -> 11.2 mm
Other:
- board text added: "3V3"
- board text added: "5V"
- board text added: "CANH"
- board text added: "CANL"
- board text added: "GND"
- board text added: "RX"
- board text added: "TX"
Changed lines of the file:
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@@
     (links 17)
     (no_connects 0)
-    (area 19.949999 19.949999 40.050001 33.050001)
+    (area 16.528972 13.65 52.035715 33.256401)
     (thickness 1.6)
-    (drawings 6)
-    (tracks 50)
+    (drawings 13)
+    (tracks 60)
     (zones 0)
     (modules 6)
@@
   (setup
     (last_trace_width 0.3302)
+    (user_trace_width 0.5)
     (trace_clearance 0.254)
     (zone_clearance 0.2032)
@@
     (visible_elements FFFFFF7F)
     (pcbplotparams
-      (layerselection 0x00030_80000001)
+      (layerselection 0x010f0_80000001)
       (usegerberextensions true)
       (excludeedgelayer true)
@@
       (psnegative false)
       (psa4output false)
-      (plotreference true)
-      (plotvalue true)
+      (plotreference false)
+      (plotvalue false)
       (plotinvisibletext false)
       (padsonsilk false)
@@
       (outputformat 1)
       (mirror false)
-      (drillshape 1)
+      (drillshape 0)
       (scaleselection 1)
       (outputdirectory ""))
@@
     )
   )
+  (gr_text CANL (at 35.687 30.1625 180) (layer B.SilkS)
+    (effects (font (size 1.5 1.5) (thickness 0.3)) (justify mirror))
+  )
+  (gr_text CANH (at 35.8775 27.559 180) (layer B.SilkS)
+    (effects (font (size 1.5 1.5) (thickness 0.3)) (justify mirror))
+  )
+  (gr_text RX (at 25.146 31.5595 180) (layer B.SilkS)
+    (effects (font (size 1.5 1.5) (thickness 0.3)) (justify mirror))
+  )
+  (gr_text TX (at 25.2095 28.8925 180) (layer B.SilkS)
+    (effects (font (size 1.5 1.5) (thickness 0.3)) (justify mirror))
+  )
+  (gr_text GND (at 25.9715 26.416 180) (layer B.SilkS)
+    (effects (font (size 1.5 1.5) (thickness 0.3)) (justify mirror))
+  )
+  (gr_text 3V3 (at 25.8826 23.876 180) (layer B.SilkS)
+    (effects (font (size 1.5 1.5) (thickness 0.3)) (justify mirror))
+  )
+  (gr_text 5V (at 25.146 21.336 180) (layer B.SilkS)
+    (effects (font (size 1.5 1.5) (thickness 0.3)) (justify mirror))
+  )
   (gr_line (start 40 33) (end 40 20) (angle 90) (layer Edge.Cuts) (width 0.1))
   (gr_line (start 20 33) (end 40 33) (angle 90) (layer Edge.Cuts) (width 0.1))
@@
   (gr_line (start 40 20) (end 20 20) (angle 90) (layer Edge.Cuts) (width 0.1))
   (dimension 13 (width 0.3) (layer Cmts.User)
-    (gr_text "13.000 mm" (at 46.1 26.5 270) (layer Cmts.User)
+    (gr_text "13.00 mm" (at 46.1 26.5 270) (layer Cmts.User)
       (effects (font (size 1.5 1.5) (thickness 0.3)))
     )
@@
   )
   (dimension 20 (width 0.3) (layer Cmts.User)
-    (gr_text "20.000 mm" (at 30 15.15) (layer Cmts.User)
+    (gr_text "20.00 mm" (at 30 15.15) (layer Cmts.User)
       (effects (font (size 1.5 1.5) (thickness 0.3)))
     )
@@
   )
   (segment (start 27.39 23.96) (end 27.4 23.97) (width 0.3556) (layer F.Cu) (net 1))
-  (segment (start 22.4 23.96) (end 27.39 23.96) (width 0.3556) (layer F.Cu) (net 1))
   (segment (start 21.8 30.3) (end 20.9 29.4) (width 0.3556) (layer F.Cu) (net 1))
   (segment (start 20.9 29.4) (end 20.9 25.46) (width 0.3556) (layer F.Cu) (net 1))
   (segment (start 20.9 25.46) (end 22.4 23.96) (width 0.3556) (layer F.Cu) (net 1))
   (segment (start 25.7 30.3) (end 21.8 30.3) (width 0.3556) (layer F.Cu) (net 1))
+  (segment (start 27.39 23.96) (end 27.4 23.97) (width 0.5) (layer F.Cu) (net 1))
+  (segment (start 22.4 23.96) (end 27.39 23.96) (width 0.5) (layer F.Cu) (net 1))
   (segment (start 27.39 21.42) (end 27.4 21.43) (width 0.3302) (layer F.Cu) (net 2))
-  (segment (start 22.4 21.42) (end 27.39 21.42) (width 0.3302) (layer F.Cu) (net 2))
+  (segment (start 27.39 21.42) (end 27.4 21.43) (width 0.5) (layer F.Cu) (net 2))
+  (segment (start 22.4 21.42) (end 27.39 21.42) (width 0.5) (layer F.Cu) (net 2))
   (segment (start 24.45 30.95) (end 23.82 31.58) (width 0.3302) (layer F.Cu) (net 3))
   (segment (start 23.82 31.58) (end 22.4 31.58) (width 0.3302) (layer F.Cu) (net 3))
@@
   (segment (start 28.246902 30.95) (end 28.3 30.896902) (width 0.3556) (layer F.Cu) (net 5))
   (segment (start 27.25 30.95) (end 28.246902 30.95) (width 0.3556) (layer F.Cu) (net 5))
-  (segment (start 35.075 25.85) (end 28.4 25.85) (width 0.3556) (layer F.Cu) (net 5))
   (segment (start 35.1 25.875) (end 35.075 25.85) (width 0.3556) (layer F.Cu) (net 5))
   (segment (start 25.85 25.85) (end 25.15 26.55) (width 0.3556) (layer F.Cu) (net 5))
-  (segment (start 28.4 25.85) (end 25.85 25.85) (width 0.3556) (layer F.Cu) (net 5))
+  (segment (start 25.2 26.5) (end 25.85 25.85) (width 0.5) (layer F.Cu) (net 5))
+  (segment (start 22.4 26.5) (end 25.2 26.5) (width 0.5) (layer F.Cu) (net 5))
+  (segment (start 25.85 25.85) (end 28.4 25.85) (width 0.5) (layer F.Cu) (net 5))
+  (segment (start 35.075 25.85) (end 35.1 25.875) (width 0.5) (layer F.Cu) (net 5))
+  (segment (start 28.4 25.85) (end 35.075 25.85) (width 0.5) (layer F.Cu) (net 5))
+  (segment (start 38.0035 22.0785) (end 38 22.075) (width 0.5) (layer F.Cu) (net 5))
+  (segment (start 38.0035 30.9215) (end 38.0035 22.0785) (width 0.5) (layer F.Cu) (net 5))
+  (segment (start 38.0035 25.875) (end 38.0035 30.9215) (width 0.5) (layer F.Cu) (net 5))
+  (segment (start 35.1 25.875) (end 38.0035 25.875) (width 0.5) (layer F.Cu) (net 5))
   (segment (start 33.175 22.7) (end 35.1 24.625) (width 0.3302) (layer F.Cu) (net 6))
-  (segment (start 27.4 22.7) (end 33.175 22.7) (width 0.3302) (layer F.Cu) (net 6))
+  (segment (start 33.175 22.7) (end 35.1 24.625) (width 0.5) (layer F.Cu) (net 6))
+  (segment (start 27.4 22.7) (end 33.175 22.7) (width 0.5) (layer F.Cu) (net 6))
   (segment (start 32.205 27.125) (end 35.1 27.125) (width 0.3302) (layer F.Cu) (net 7))
   (segment (start 31.6 27.73) (end 32.205 27.125) (width 0.3302) (layer F.Cu) (net 7))
